File: pcb/bauble_pcb.kicad_sch (KiCad schematic)
At the start: 19 parts, among them J1 Conn_01x02, J2 Conn_01x04, J3 Conn_01x02, J4 Conn_01x02, Q1 AO3401, U1 HT7833_SOT89, U2 TP4057, U3 ESP32-C3-WROOM-02

Commit message: Exclude connectors in schematic from BOM
Parts:
- J1, J2, J3, J4: now left out of the parts list
Changed lines of the file:
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@@
   )
   (symbol (lib_id "Connector_Generic:Conn_01x02") (at 99.06 96.52 180) (unit 1)
-    (in_bom yes) (on_board yes)
+    (in_bom no) (on_board yes)
     (property "Reference" "J1" (id 0) (at 90.17 90.17 0))
     (property "Value" "Conn_01x02" (id 1) (at 90.17 92.71 0))
@@
   )
   (symbol (lib_id "Connector_Generic:Conn_01x04") (at 179.07 78.74 0) (unit 1)
-    (in_bom yes) (on_board yes) (fields_autoplaced)
+    (in_bom no) (on_board yes) (fields_autoplaced)
     (property "Reference" "J2" (id 0) (at 181.102 79.1753 0)
       (effects (font (size 1.27 1.27)) (justify left))
@@
   )
   (symbol (lib_id "Connector_Generic:Conn_01x02") (at 113.03 144.78 270) (unit 1)
-    (in_bom yes) (on_board yes) (fields_autoplaced)
+    (in_bom no) (on_board yes) (fields_autoplaced)
     (property "Reference" "J4" (id 0) (at 115.062 143.9453 90)
       (effects (font (size 1.27 1.27)) (justify left))
@@
   )
   (symbol (lib_id "Connector_Generic:Conn_01x02") (at 96.52 146.05 0) (unit 1)
-    (in_bom yes) (on_board yes) (fields_autoplaced)
+    (in_bom no) (on_board yes) (fields_autoplaced)
     (property "Reference" "J3" (id 0) (at 98.552 146.4853 0)
       (effects (font (size 1.27 1.27)) (justify left))

Commit message: Remove LCD and ESP32 from BOM
Parts:
- DISP1, U3: now left out of the parts list
Changed lines of the file:
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@@
   )
   (symbol (lib_id "Espressif:ESP32-C3-WROOM-02") (at 130.81 87.63 0) (unit 1)
-    (in_bom yes) (on_board yes) (fields_autoplaced)
+    (in_bom no) (on_board yes) (fields_autoplaced)
     (property "Reference" "U3" (id 0) (at 131.445 52.3072 0))
     (property "Value" "ESP32-C3-WROOM-02" (id 1) (at 131.445 54.8441 0))
@@
   )
   (symbol (lib_id "Jeroens lib:LCD_LH096T") (at 219.71 96.52 0) (unit 1)
-    (in_bom yes) (on_board yes) (fields_autoplaced)
+    (in_bom no) (on_board yes) (fields_autoplaced)
     (property "Reference" "DISP1" (id 0) (at 230.505 98.8603 0)
       (effects (font (size 1.27 1.27)) (justify left))
@@
   (symbol (lib_id "power:+3V3") (at 91.44 76.2 0) (unit 1)
     (in_bom yes) (on_board yes) (fields_autoplaced)
-    (property "Reference" "#PWR?" (id 0) (at 91.44 80.01 0)
+    (property "Reference" "#PWR0118" (id 0) (at 91.44 80.01 0)
       (effects (font (size 1.27 1.27)) hide)
     )
@@
     )
     (path "/9cad33bf-0dc9-4e38-8ef0-2a0030389af7"
-      (reference "#PWR?") (unit 1) (value "+3V3") (footprint "")
+      (reference "#PWR0118") (unit 1) (value "+3V3") (footprint "")
     )
     (path "/305fe303-2dc1-4958-b9c7-868442bbd927"
